File: pcb/smeat/v1/esp32-wroom-timer/esp32-wroom-timer.kicad_pcb (KiCad board)
At the start: 2 copper layers, 49.5 x 51.2 mm, 56 parts, among them J1 Fan_connector, J2 Conn_01x06_Male, J3 input power, Q1 Q_NMOS_GSD, Q2 Q_NMOS_GSD, U1 ESP32-WROOM-32, U2 AMS1117, U3 RX5808, U4 MP1584, U5 RX5808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

Commit message: Final(?) version of PCB
Parts:
- moved C15 0.21 mm to (72.5, 66.1)
- moved C11 0.13 mm to (70.6, 66.1)
Routing:
- net +5V: track 96.7 -> 103.5 mm, vias 8 -> 10
- net /CLK: track 72.9 -> 67.0 mm
- net GND: track 88.6 -> 83.3 mm, vias 30 -> 207
- net +28V: track 16.8 -> 19.8 mm
- net /RTS: track 41.4 -> 40.6 mm
- net /V_SENSE: vias 0 -> 2
