File: pcb/smeat/esp32-wroom-timer-v1/esp32-wroom-timer.kicad_pcb (KiCad board)
At the start: 2 copper layers, 74.4 x 51.2 mm, 62 parts, among them J1 Fan_connector, J2 Programming, J3 input power, J4 Conn_Coaxial, Q1 Q_NMOS_GSD, Q2 Q_NMOS_GSD, U1 ESP32-WROOM-32U, U10 RX5808, U11 RX5808, U12 MCP9804_MSOP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

Commit message: Possibly the final version(?)
Parts:
- D2: footprint Diode_SMD:D_SOD-123 -> Diode_SMD:D_SMA
- R6, R7: moved to B.Cu
- moved R7 6.92 mm to (94.6, 77.4), turned to 180 degrees
- moved R6 0.75 mm to (91.4, 77.4), turned to 180 degrees
- moved D2 0.25 mm to (69.2, 59.2)
Connections:
- R6 pad 1: /ADC6 -> /ADC5
- R7 pad 2: /ADC6 -> /ADC5
Routing:
- net /ADC6: track 52.1 -> 47.0 mm
- net /ADC5: track 51.1 -> 55.6 mm
- net GND: track 75.5 -> 71.6 mm, vias 351 -> 350
- net +5V: track 121.0 -> 118.4 mm
- net /CS1: track 18.3 -> 15.9 mm
- net /CS3: track 59.2 -> 60.9 mm
- net /CS4: track 41.7 -> 40.4 mm, vias 2 -> 0
- net /CLK: track 90.4 -> 89.1 mm, vias 5 -> 6
- net +28V: track 26.3 -> 27.1 mm, vias 3 -> 4
- net Net-(D2-Pad2): track 8.80 -> 9.40 mm
- net /SDA: track 58.9 -> 59.5 mm
- net /CS5: track 78.7 -> 78.4 mm, vias 2 -> 0
- net /MOSI: track 109.9 -> 110.2 mm, vias 4 -> 5
- net Net-(Q1-Pad1): track 1.73 -> 1.74 mm, vias 2 -> 1
